Commit message: Split odometry launches out of mapping; add bag static TF
Renames fastlio_mapping/pointlio_mapping launches to *_odometry and adds
dec_launch/launch/bag_static_tf.launch.py, reconstructing the rig's
static transforms for bag replay.

NOTE for bag replay: pepper_sensor_tf.launch.py needs scope:=all. The
default 'mount' scope omits the owner:driver camera edges on the
assumption the RealSense driver is publishing them live; with no driver
the tree comes up as three disconnected islands and every consumer that
looks up base_footprint silently produces nothing.

File: pepper_slam/urdf/sensor_rig.xacro (robot description, xacro)
@@ -64,5 +64,12 @@
       <parent link="l2lidar_frame"/>
       <child  link="camera_camera_link"/>
-      <origin xyz="0.038508 -0.036458 0.012712" rpy="-0.464105854 -1.544163393 -3.127486964"/>
+      <!-- KEEP IN SYNC WITH config/sensor_tf.yaml. This is the same physical
+           transform expressed twice: the YAML publishes it to /tf_static, this
+           joint only positions the meshes for visualisation. They drifted once
+           already (rotation measured 2026-08-06 and updated in the YAML while
+           this still held the old inherited value), so a rig view can silently
+           show geometry the robot is not using. Equivalent quaternion:
+           qxyzw [0.674794, -0.166617, 0.703353, 0.148951] -->
+      <origin xyz="0.038541 -0.036473 0.021032" rpy="-0.779068046 -1.523300726 -2.812723308"/>
     </joint>
     <!-- The RealSense's OWN internal extrinsics. realsense2_camera publishes
